File: ethernet chip.sch (EAGLE design)
At the start: 29 parts

Commit message: Updated Ethernet Schematic (Paul)
Parts:
- removed C10, C7, C8, C9: (no value), eagle-ltspice:CC0603
- added R19, R20: 27R, resistor:R-US_R0603
- added R8: 10K, SparkFun-Passives:RESISTOR0603-RES
- added U$2: J00-0065NL, Paul's Library:J00-0065NL
- added U$3: ECX-32, Other:ECX-32
- added U$4: (no value), EthernetChip:553-2382-1-ND
- C1, C2: value (none) -> 22pF/50V
- C3: value (none) -> 2.2uF/10V
- C4, C5, C6: value (none) -> 100nF/25V
- R1, R15, R2, R3, R4, R5, R6, R7: value (none) -> 27R; device eagle-ltspice:RR0603 -> resistor:R-US_R0603
- R10, R9: value (none) -> 250R; device eagle-ltspice:RR0603 -> resistor:R-US_R0603
- R11, R12, R13, R14: value (none) -> 49.9R; device eagle-ltspice:RR0603 -> resistor:R-US_R0603
- R16: value (none) -> 1M; device eagle-ltspice:RR0603 -> resistor:R-US_R0603
- R17: value (none) -> 12.1K; device eagle-ltspice:RR0603 -> resistor:R-US_R0603
- R18: value (none) -> 10K; device eagle-ltspice:RR0603 -> resistor:R-US_R0603
Connections:
- removed net N$13: C2.1, R9.1, U$1.XTAL1/CLKIN
- removed net N$6: C1.2, R9.2, U$1.XTAL2
- new net BUS_SPEED: R18.2, U$1.LED2/NINTSEL, U$2.G_GND
- new net CRSDV: R3.1
- new net CT1: C5.2, C6.2, R11.2, R12.2, R13.2, R14.2, U$2.CT1, U$2.CT2
- new net GREEN: R9.2, U$2.G
- new net LINK/ACT: U$1.LED1/REGOFF, U$2.Y
- new net MDE: R15.2, U$1.MDC
- new net MDIO: R19.2, U$1.MDIO
- new net RD+: R13.1, U$1.RXP, U$2.RD+
- new net RD-: R14.1, U$1.RXN, U$2.RD-
- new net REFCLK: R4.1
- new net RXD1: R2.1
- new net RXDO: R1.1
- new net RXERR: U$1.RXER/PHYAD0
- new net TD+: R11.1, U$1.TXP, U$2.TD+
- new net TD-: R12.1, U$1.TXN, U$2.TD-
- new net TXD0: R6.1
- new net TXD1: R7.1
- new net TXEN: R5.1
- new net XTAL1: C2.1, R16.1, U$1.XTAL1/CLKIN, U$3.OUT/IN
- new net XTAL2: C1.1, R16.2, U$1.XTAL2, U$3.IN/OUT
- new net YELLOW: R10.2, U$2.Y_GND
- net +3V3: now also R10.1, R8.2, R9.1, U$4.2; no longer C10.1, C5.2, C6.2, C7.1, C8.1, C9.1, R11.2, R12.2, R13.2, R14.2, R15.2, R16.2, R17.2
- net GND: now also C1.2, R17.1, U$2.CHS1, U$2.CHS2, U$2.GND, U$3.GND1, U$3.GND2; no longer C1.1, C10.2, C7.2, C8.2, C9.2, R10.2
- net N$11: now also U$4.1; no longer R11.1
- net N$14: now also R8.1, U$1.NRST; no longer R18.2, U$1.LED2/NINTSEL
- net N$4: now also R17.2; no longer R10.1
Other:
- moved on the sheet: C1, C2, C5, C6
